Commit message: visualize the carmodel in rviz

File: ros2_ws/src/mentorpi_description/urdf/ack.xacro (robot description, xacro)
@@ -149,5 +149,5 @@
     <axis xyz="-2.2787E-05 1 1.9439E-05"/>
   </joint>
-  <link name="depth_cam">
+  <link name="camera_link">
     <inertial>
       <origin rpy="0 0 0" xyz="0.0023402290651429 0.00113784597946548 -0.0102127064032341"/>
@@ -174,5 +174,5 @@
     <origin rpy="0 0 0" xyz="0.064015 -0.00013463 0.051155"/>
     <parent link="base_link"/>
-    <child link="depth_cam"/>
+    <child link="camera_link"/>
     <axis xyz="0 0 0"/>
   </joint>
